File: Projet_capteur_pcb/Projet_capteur_pcb.kicad_pcb (KiCad board)
At the start: 2 copper layers, 68.6 x 53.3 mm, 22 parts, among them J1 Power, J2 Digital/PWM, J3 Analog, J4 Digital/PWM

Commit message: 3D + placement
Parts:
- C1, C2, C3: footprint Capacitor_THT:C_Disc_D10.5mm_W5.0mm_P5.00mm -> Capacitor_THT:C_Disc_D7.5mm_W2.5mm_P5.00mm
- moved C1 38.9 mm to (114.0, 87.0)
- moved C2 33.8 mm to (115.0, 92.5)
- moved EcranOled1 31.3 mm to (145.0, 84.5)
- moved R4 27.8 mm to (132.0, 80.7)
- moved R5 21.2 mm to (112.1, 53.0)
- moved R1 18.7 mm to (108.5, 80.2)
- moved C3 18.4 mm to (103.5, 76.5)
- moved Encodeur1 15.8 mm to (162.0, 60.6), turned to -90 degrees
- moved Bluetooth1 11.3 mm to (148.7, 54.5), turned to 0 degrees
- moved R3 11.2 mm to (127.0, 80.6)
- moved aop 10.7 mm to (130.3, 89.3)
- moved C4 10.2 mm to (114.0, 77.5)
- moved potD1 1.92 mm to (118.7, 63.2)
- moved REF** 1.12 mm to (166.0, 83.0)
Routing:
- added copper zone on B.Cu, net GND
