File: Projet_capteur_pcb/Projet_capteur_pcb.kicad_sch (KiCad schematic)
At the start: 18 parts, among them J1 Power, J2 Digital/PWM, J3 Analog, J4 Digital/PWM

Commit message: 3D + placement
Parts:
- C1, C2, C3: footprint Capacitor_THT:C_Disc_D10.5mm_W5.0mm_P5.00mm -> Capacitor_THT:C_Disc_D7.5mm_W2.5mm_P5.00mm
Changed lines of the file:
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@@
 			)
 		)
-		(property "Footprint" "Capacitor_THT:C_Disc_D10.5mm_W5.0mm_P5.00mm"
+		(property "Footprint" "Capacitor_THT:C_Disc_D7.5mm_W2.5mm_P5.00mm"
 			(at 146.05 136.8552 0)
 			(effects
@@
 			)
 		)
-		(property "Footprint" "Capacitor_THT:C_Disc_D10.5mm_W5.0mm_P5.00mm"
+		(property "Footprint" "Capacitor_THT:C_Disc_D7.5mm_W2.5mm_P5.00mm"
 			(at 275.59 124.7648 0)
 			(effects
@@
 			)
 		)
-		(property "Footprint" "Capacitor_THT:C_Disc_D10.5mm_W5.0mm_P5.00mm"
+		(property "Footprint" "Capacitor_THT:C_Disc_D7.5mm_W2.5mm_P5.00mm"
 			(at 190.1952 147.32 0)
 			(effects
